Commit message: Imported upstream version '0.1.1' of 'upstream'

File: barrett_hand_description/robots/bh_alone.urdf.xacro (robot description, xacro)
@@ -2,5 +2,5 @@
 <robot name="bhand" xmlns:xacro="http://www.ros.org/wiki/xacro">
 	<!-- Available choices: bh282.urdf.xacro, bh280.urdf.xacro -->
-	<xacro:include filename="$(find barrett_hand_description)/urdf/bh282.urdf.xacro" />
+	<xacro:include filename="$(find barrett_hand_description)/urdf/bh280.urdf.xacro" />
 	<!-- z-coordinate is not 0 because otherwise the hand base tilts when the simulation is started -->
 	<link name="base_link">
@@ -27,3 +27,10 @@
 		<origin xyz="0 0 0" rpy="0 0 0" />
 	</xacro:bhand_macro>
+	<gazebo>
+	    <plugin name="ros_control" filename="libgazebo_ros_control.so">
+	       <robotNamespace>/</robotNamespace>
+	       <controlPeriod>0.001</controlPeriod>
+	       <robotSimType>gazebo_ros_control/DefaultRobotHWSim</robotSimType>
+	    </plugin>
+    </gazebo>
 </robot>

File: barrett_hand_description/urdf/bh280.urdf.xacro (robot description, xacro)
@@ -1,4 +1,4 @@
 <?xml version="1.0"?>
-<robot xmlns:xacro="http://www.ros.org/wiki/xacro">
+<robot xmlns:xacro="http://ros.org/wiki/xacro">
 	<!-- Import all Gazebo-customization elements, including Gazebo colors -->
 	<xacro:include filename="$(find barrett_hand_description)/urdf/bh282.gazebo.xacro" />
@@ -13,5 +13,5 @@
 	<xacro:macro name="bhand_macro" params="parent name *origin">
 		<joint name="${name}_base_joint" type="fixed">
-			<insert_block name="origin"/>
+			<xacro:insert_block name="origin"/>
 			<parent link="${parent}"/>
 			<child link="${name}_base_link"/>
@@ -112,4 +112,5 @@
 			<origin xyz="-0.069936 0.003 0" rpy="0 0 0" />
 			<axis xyz="0 0 -1"/>
+			<mimic joint="${name}_j32_joint" multiplier="${0.84/2.44}" />
 			<limit effort="${joint_effort_limit}" lower="0.0" upper="0.84" velocity="${joint_velocity_limit}"/>
 			<dynamics damping="${joint_damping}" friction="${joint_friction}"/>
@@ -239,4 +240,5 @@
 			<origin xyz="-0.069936 0.003 0" rpy="0 0 0" />
 			<axis xyz="0 0 -1"/>
+			<mimic joint="${name}_j12_joint" multiplier="${0.84/2.44}" />
 			<limit effort="${joint_effort_limit}" lower="0.0" upper="0.84" velocity="${joint_velocity_limit}"/>
 			<dynamics damping="${joint_damping}" friction="${joint_friction}"/>
@@ -281,4 +283,5 @@
 			<origin xyz="-0.025 0 0.0415" rpy="0 0 -1.5708" />
 			<axis xyz="0 0 1"/>
+			<mimic joint="${name}_j11_joint" multiplier="1" />
 			<limit effort="${joint_effort_limit}" lower="0" upper="3.1416" velocity="${joint_velocity_limit}"/>
 			<dynamics damping="${joint_damping}" friction="${joint_friction}"/>
@@ -366,4 +369,5 @@
 			<origin xyz="-0.069936 0.003 0" rpy="0 0 0" />
 			<axis xyz="0 0 -1"/>
+			<mimic joint="${name}_j22_joint" multiplier="${0.84/2.44}" />
 			<limit effort="${joint_effort_limit}" lower="0.0" upper="0.84" velocity="${joint_velocity_limit}"/>
 			<dynamics damping="${joint_damping}" friction="${joint_friction}"/>

File: barrett_hand_description/urdf/bh282.gazebo.xacro (robot description, xacro)
@@ -2,16 +2,8 @@
 <robot xmlns:xacro="http://ros.org/wiki/xacro">
   <xacro:macro name="bh_gazebo" params="name">
-	<!-- ros_control plugin -->
-	<gazebo>
-		<plugin name="ros_control" filename="libgazebo_ros_control.so">
-		   <robotNamespace>/</robotNamespace>
-		   <controlPeriod>0.001</controlPeriod>
-		   <robotSimType>gazebo_ros_control/DefaultRobotHWSim</robotSimType>
-		</plugin>
-	</gazebo>
 	<gazebo>
 	   	<plugin name="mimic_plugin" filename="libgazebo_mimic_plugin.so">
-       		   <joint>bh_j11_joint</joint>
-       		   <mimicJoint>bh_j21_joint</mimicJoint>
+       		   <joint>${name}_j11_joint</joint>
+       		   <mimicJoint>${name}_j21_joint</mimicJoint>
        		   <multiplier>1</multiplier>
        		</plugin>
@@ -19,6 +11,6 @@
 	<gazebo>
 	    	<plugin name="mimic_plugin" filename="libgazebo_mimic_plugin.so">
-       		   <joint>bh_j12_joint</joint>
-       		   <mimicJoint>bh_j13_joint</mimicJoint>
+       		   <joint>${name}_j12_joint</joint>
+       		   <mimicJoint>${name}_j13_joint</mimicJoint>
        		   <multiplier>0.344</multiplier>
        		</plugin>
@@ -26,6 +18,6 @@
 	<gazebo>
 	    	<plugin name="mimic_plugin" filename="libgazebo_mimic_plugin.so">
-       		   <joint>bh_j22_joint</joint>
-       		   <mimicJoint>bh_j23_joint</mimicJoint>
+       		   <joint>${name}_j22_joint</joint>
+       		   <mimicJoint>${name}_j23_joint</mimicJoint>
        		   <multiplier>0.344</multiplier>
        		</plugin>
@@ -33,6 +25,6 @@
 	<gazebo>
 	    	<plugin name="mimic_plugin" filename="libgazebo_mimic_plugin.so">
-       		   <joint>bh_j32_joint</joint>
-       		   <mimicJoint>bh_j33_joint</mimicJoint>
+       		   <joint>${name}_j32_joint</joint>
+       		   <mimicJoint>${name}_j33_joint</mimicJoint>
        		   <multiplier>0.344</multiplier>
        		</plugin>
